Commit message: foundation is complete for diff drive

File: rover_description/meshes/Assem10.urdf (robot description, URDF)
Before this commit: robot Assem10, 17 links, 16 joints
Links:
- removed link CAM_FL
- removed link CAM_FR
- removed link CAM_FRONT
- removed link CAM_LEFT
- removed link CAM_REAR
- removed link CAM_RIGHT
- removed link CAM_SCIENCE
- added link Front_Cam1, mass 0.0146410874338426; visual mesh filename=package://rover_description/meshes/GPS.STL
- added link Front_Cam2, mass 0.0146410874338426; visual mesh filename=package://rover_description/meshes/GPS.STL
Joints:
- removed joint CAM_FL_joint
- removed joint CAM_FRONT_joint
- removed joint CAM_FR_joint
- removed joint CAM_LEFT_joint
- removed joint CAM_REAR_joint
- removed joint CAM_RIGHT_joint
- removed joint CAM_SCIENCE_joint
