Commit message: description package fixed

File: rover_description/urdf/Assem10.urdf (robot description, URDF)
Before this commit: robot Assem10, 9 links, 8 joints
Links:
- added link chassis_link, mass 9.90010001726695; collision mesh filename=package://rover_description/meshes/base_link.STL; visual mesh filename=package://rover_description/meshes/base_link.STL
- link base_link: mass 9.90010001726695 -> None; geometry 
Joints:
- added joint base_to_chassis_joint: type fixed, parent base_link, child chassis_link, origin xyz=0 0 0.4 rpy=0 -1.5708 0
- joint FLOW_CAM_joint: parent base_link -> chassis_link
- joint GPS_joint: parent base_link -> chassis_link
- joint IMU_joint: parent base_link -> chassis_link
- joint LB_joint: parent base_link -> chassis_link
- joint LF_joint: parent base_link -> chassis_link
- joint OPTICAL_joint: parent base_link -> chassis_link
- joint RB_joint: parent base_link -> chassis_link
- joint RF_joint: parent base_link -> chassis_link

File: rover_description/urdf/Assem10_real.urdf.xacro (robot description, xacro)
@@ -3,5 +3,5 @@
   Assem10_real.urdf.xacro
   Real-hardware variant of the rover URDF.
-  Replaces IgnitionSystem with RoverCANInterface for ros2_control.
+  Replaces IgnitionSystem with RoverSerialInterface for ros2_control.
   All geometry, joints, and sensors are inherited from Assem10.urdf via xacro:include.
 -->
@@ -9,11 +9,11 @@
   <!-- Pull in the base URDF (geometry, sensors, TF tree) -->
   <xacro:include filename="$(find rover_description)/urdf/Assem10.urdf"/>
-  <!-- Override the ros2_control hardware plugin: replace IgnitionSystem with real CAN interface -->
+  <!-- Override the ros2_control hardware plugin: replace IgnitionSystem with real UART interface -->
   <!-- NOTE: This replaces the <ros2_control> block defined in Assem10.urdf at load time.
        ros2_control_node will use the *last* matching block it finds in the merged model. -->
   <ros2_control name="RoverRealSystem" type="system">
     <hardware>
-      <plugin>rover_hardware/RoverCANInterface</plugin>
-      <param name="can_interface">can0</param>
+      <plugin>rover_hardware/RoverSerialInterface</plugin>
+      <param name="serial_port">/dev/ttyTHS0</param>
     </hardware>
     <joint name="LF_joint">
@@ -22,10 +22,10 @@
       <state_interface name="velocity"/>
     </joint>
-    <joint name="RF_joint">
+    <joint name="LB_joint">
       <command_interface name="velocity"/>
       <state_interface name="position"/>
       <state_interface name="velocity"/>
     </joint>
-    <joint name="LB_joint">
+    <joint name="RF_joint">
       <command_interface name="velocity"/>
       <state_interface name="position"/>

Commit message: enviorment-setup

File: rover_description/urdf/Assem10.urdf (robot description, URDF)
Before this commit: robot Assem10, 17 links, 16 joints
Links:
- link LB: geometry collision cylinder length=0.08 radius=0.14; visual mesh filename=package://rover_description/meshes/LB.STL
- link LF: geometry collision cylinder length=0.08 radius=0.14; visual mesh filename=package://rover_description/meshes/LF.STL
- link RB: geometry collision cylinder length=0.08 radius=0.14; visual mesh filename=package://rover_description/meshes/RB.STL
- link RF: geometry collision cylinder length=0.08 radius=0.14; visual mesh filename=package://rover_description/meshes/RF.STL
