Commit message: added dome_insider

File: rover_description/urdf/Assem10.urdf (robot description, URDF)
Before this commit: robot Assem10, 18 links, 17 joints
Joints:
- joint OPTICAL_joint: origin xyz=-0.091551 0.0046556 0.087323 rpy=-1.5708 0 -1.5708 -> xyz=0.28 0.0046556 0.18 rpy=-1.5708 0 -1.5708
