Commit message: Updated rover urdf

File: rover_description/urdf/rarm.urdf (robot description, URDF)
Before this commit: robot rover_with_arm, 28 links, 27 joints
Joints:
- joint CAM_FL_joint: origin xyz=0.07 0.20 -0.18 rpy=-0.7854 0 0 -> xyz=0.07 0.20 -0.18 rpy=1.5708 0.7854 1.5708
- joint CAM_FRONT_joint: origin xyz=0.07 0.0 -0.22 rpy=-1.5708 0 -1.5708 -> xyz=0.07 0.0 -0.22 rpy=0 1.5708 0
- joint CAM_FR_joint: origin xyz=0.07 -0.20 -0.18 rpy=-0.7854 0 3.1416 -> xyz=0.07 -0.20 -0.18 rpy=-1.5708 0.7854 -1.5708
- joint CAM_LEFT_joint: origin xyz=0.04 0.26 0.15 rpy=0 0 0 -> xyz=0.04 0.26 0.15 rpy=1.5708 0 1.5708
- joint CAM_REAR_joint: origin xyz=0.07 0.0 0.28 rpy=1.5708 0 0 -> xyz=0.07 0.0 0.28 rpy=0 -1.5708 -3.1416
- joint CAM_RIGHT_joint: origin xyz=0.04 -0.26 0.15 rpy=0 0 3.1416 -> xyz=0.04 -0.26 0.15 rpy=-1.5708 0 -1.5708
- joint LB_joint: limit effort=100 velocity=10 -> effort=1000 velocity=10
- joint LF_joint: limit effort=100 velocity=10 -> effort=1000 velocity=10
- joint RB_joint: limit effort=100 velocity=10 -> effort=1000 velocity=10
- joint RF_joint: limit effort=100 velocity=10 -> effort=1000 velocity=10

Commit message: updated urdf

File: rover_description/urdf/rarm.urdf (robot description, URDF)
Before this commit: robot rover_with_arm, 28 links, 27 joints
Joints:
- joint CAM_FL_joint: origin xyz=0.07 0.20 -0.18 rpy=1.5708 0.7854 1.5708 -> xyz=0.07 0.20 -0.18 rpy=-1.5708 -0.7854 -1.5708
- joint CAM_FRONT_joint: origin xyz=0.07 0.0 -0.22 rpy=0 1.5708 0 -> xyz=0.07 0.0 -0.22 rpy=-1.5708 0 -1.5708
- joint CAM_LEFT_joint: origin xyz=0.04 0.26 0.15 rpy=1.5708 0 1.5708 -> xyz=0.04 0.26 0.15 rpy=0 1.5708 0
- joint CAM_REAR_joint: origin xyz=0.07 0.0 0.28 rpy=0 -1.5708 -3.1416 -> xyz=0.07 0.0 0.28 rpy=1.5708 0 1.5708
- joint CAM_RIGHT_joint: origin xyz=0.04 -0.26 0.15 rpy=-1.5708 0 -1.5708 -> xyz=0.04 -0.26 0.15 rpy=0 -1.5708 -3.1416
- joint CAM_SCIENCE_joint: origin xyz=-0.12 0.0 -0.20 rpy=0 0 1.5708 -> xyz=-0.12 0.0 -0.20 rpy=-1.5708 0 -1.5708

Commit message: updated urdf v2

File: rover_description/urdf/rarm.urdf (robot description, URDF)
Before this commit: robot rover_with_arm, 28 links, 27 joints
Links:
- removed link arm_base_link
- added link gripper_rgbd_camera, mass 0.05; collision box size=0.07 0.04 0.05; visual box size=0.07 0.002 0.014
Joints:
- removed joint rover_to_arm_joint
- added joint gripper_rgbd_camera_joint: type fixed, parent gripper-base, child gripper_rgbd_camera, origin xyz=0.0 0.02 0.05 rpy=1.34 0 -1.30
- joint z_axis: origin xyz=0.0211020680489503 0.0649999999999998 0.0950000000000002 rpy=0 0 0 -> xyz=0.12 0.05 -0.02 rpy=0 1.57 0; parent arm_base_link -> chassis_link

Commit message: updated urdf

File: rover_description/urdf/rarm.urdf (robot description, URDF)
Before this commit: robot rover_with_arm, 28 links, 27 joints
Joints:
- joint gripper-wrist: limit (none) -> lower=-1.57 upper=1.57 effort=100 velocity=10; type continuous -> revolute
- joint gripper_rgbd_camera_joint: origin xyz=0.0 0.02 0.05 rpy=1.34 0 -1.30 -> xyz=0.0 -0.05 0.05 rpy=3.14 0 -1.57

Commit message: updated urdf

File: rover_description/urdf/rarm.urdf (robot description, URDF)
Before this commit: robot rover_with_arm, 28 links, 27 joints
Joints:
- joint gripper_rgbd_camera_joint: origin xyz=0.0 -0.05 0.05 rpy=3.14 0 -1.57 -> xyz=0.0 -0.10 0.05 rpy=3.14 0 -1.57

Commit message: Update

File: rover_description/urdf/rarm.urdf (robot description, URDF)
Before this commit: robot rover_with_arm, 28 links, 27 joints
Links:
- link LB: geometry collision cylinder length=0.152 radius=0.126; visual mesh filename=package://rover_description/meshes/LB.STL
- link LF: geometry collision cylinder length=0.152 radius=0.126; visual mesh filename=package://rover_description/meshes/LF.STL
- link RB: geometry collision cylinder length=0.152 radius=0.126; visual mesh filename=package://rover_description/meshes/RB.STL
- link RF: geometry collision cylinder length=0.152 radius=0.126; visual mesh filename=package://rover_description/meshes/RF.STL

Commit message: update

File: rover_description/urdf/rarm.urdf (robot description, URDF)
Before this commit: robot rover_with_arm, 28 links, 27 joints
Links:
- link LB: geometry collision mesh filename=package://rover_description/meshes/LB.STL; visual mesh filename=package://rover_description/meshes/LB.STL
- link LF: geometry collision mesh filename=package://rover_description/meshes/LF.STL; visual mesh filename=package://rover_description/meshes/LF.STL
- link RB: geometry collision mesh filename=package://rover_description/meshes/RB.STL; visual mesh filename=package://rover_description/meshes/RB.STL
- link RF: geometry collision mesh filename=package://rover_description/meshes/RF.STL; visual mesh filename=package://rover_description/meshes/RF.STL

Commit message: Added new IK control system

File: rover_description/urdf/rarm.urdf (robot description, URDF)
Before this commit: robot rover_with_arm, 28 links, 27 joints
Joints:
- joint link_1: limit lower=-0.52 upper=0.62 effort=100 velocity=10 -> lower=-0.52 upper=0.96 effort=100 velocity=10
